File: pinball_trough_transmitter.A-18617.kicad_pcb (KiCad board)
At the start: 2 copper layers, 162.6 x 88.5 mm, 16 parts, among them J1 Conn_01x09_Male, J2 Conn_01x09_Male, Q1 SFH460, Q2 SFH460, Q3 SFH460, Q4 SFH460, Q5 SFH460, Q6 SFH460, Q7 SFH460

Commit message: Minor adjustments
Parts:
- moved D7 1.27 mm to (76.8, 59.7)
- moved D6 1.02 mm to (103.9, 62.2)
- moved D5 0.76 mm to (130.9, 64.8)
- moved D4 0.51 mm to (158.0, 67.3)
- moved D3 0.25 mm to (185.0, 69.8)
Changed lines of the file:
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@@
   )
   (module LED_THT:LED_D5.0mm_Clear (layer F.Cu)
-    (at 75.565 59.69 270)
+    (at 76.835 59.69 270)
     (descr "LED, diameter 5.0mm, 2 pins, http://cdn-reichelt.de/documents/datenblatt/A500/LL-504BC2E-009.pdf")
     (tags "LED diameter 5.0mm 2 pins")
@@
   )
   (module LED_THT:LED_D5.0mm_Clear (layer F.Cu)
-    (at 102.87 62.23 270)
+    (at 103.886 62.23 270)
     (descr "LED, diameter 5.0mm, 2 pins, http://cdn-reichelt.de/documents/datenblatt/A500/LL-504BC2E-009.pdf")
     (tags "LED diameter 5.0mm 2 pins")
@@
   )
   (module LED_THT:LED_D5.0mm_Clear (layer F.Cu)
-    (at 130.175 64.77 270)
+    (at 130.937 64.77 270)
     (descr "LED, diameter 5.0mm, 2 pins, http://cdn-reichelt.de/documents/datenblatt/A500/LL-504BC2E-009.pdf")
     (tags "LED diameter 5.0mm 2 pins")
@@
   )
   (module LED_THT:LED_D5.0mm_Clear (layer F.Cu)
-    (at 157.48 67.31 270)
+    (at 157.988 67.31 270)
     (descr "LED, diameter 5.0mm, 2 pins, http://cdn-reichelt.de/documents/datenblatt/A500/LL-504BC2E-009.pdf")
     (tags "LED diameter 5.0mm 2 pins")
@@
   )
   (module LED_THT:LED_D5.0mm_Clear (layer F.Cu)
-    (at 184.785 69.85 270)
+    (at 185.039 69.85 270)
     (descr "LED, diameter 5.0mm, 2 pins, http://cdn-reichelt.de/documents/datenblatt/A500/LL-504BC2E-009.pdf")
     (tags "LED diameter 5.0mm 2 pins")
@@
   (gr_line (start 208.28 69.85) (end 208.28 77.47) (layer F.SilkS) (width 0.15))
   (gr_line (start 215.9 69.85) (end 208.28 69.85) (layer F.SilkS) (width 0.15))
-  (gr_line (start 180.975 67.31) (end 180.975 74.93) (layer F.SilkS) (width 0.15))
-  (gr_line (start 188.595 67.31) (end 180.975 67.31) (layer F.SilkS) (width 0.15))
-  (gr_line (start 153.67 64.77) (end 153.67 72.39) (layer F.SilkS) (width 0.15))
-  (gr_line (start 161.29 64.77) (end 153.67 64.77) (layer F.SilkS) (width 0.15))
-  (gr_line (start 126.365 62.23) (end 126.365 69.85) (layer F.SilkS) (width 0.15))
-  (gr_line (start 133.985 62.23) (end 126.365 62.23) (layer F.SilkS) (width 0.15))
-  (gr_line (start 99.06 59.69) (end 99.06 67.31) (layer F.SilkS) (width 0.15))
-  (gr_line (start 106.68 59.69) (end 99.06 59.69) (layer F.SilkS) (width 0.15))
-  (gr_line (start 71.755 57.15) (end 71.755 64.77) (layer F.SilkS) (width 0.15))
-  (gr_line (start 79.375 57.15) (end 71.755 57.15) (layer F.SilkS) (width 0.15))
+  (gr_line (start 181.229 67.31) (end 181.229 74.93) (layer F.SilkS) (width 0.15))
+  (gr_line (start 188.849 67.31) (end 181.229 67.31) (layer F.SilkS) (width 0.15))
+  (gr_line (start 154.178 64.77) (end 154.178 72.39) (layer F.SilkS) (width 0.15))
+  (gr_line (start 161.798 64.77) (end 154.178 64.77) (layer F.SilkS) (width 0.15))
+  (gr_line (start 127.127 62.23) (end 127.127 69.85) (layer F.SilkS) (width 0.15))
+  (gr_line (start 134.747 62.23) (end 127.127 62.23) (layer F.SilkS) (width 0.15))
+  (gr_line (start 100.076 59.69) (end 100.076 67.31) (layer F.SilkS) (width 0.15))
+  (gr_line (start 107.696 59.69) (end 100.076 59.69) (layer F.SilkS) (width 0.15))
+  (gr_line (start 73.025 57.15) (end 73.025 64.77) (layer F.SilkS) (width 0.15))
+  (gr_line (start 80.645 57.15) (end 73.025 57.15) (layer F.SilkS) (width 0.15))
   (gr_circle (center 144.145 57.785) (end 145.632898 59.055) (layer Edge.Cuts) (width 0.15))
   (gr_circle (center 90.17 59.69) (end 91.657898 60.96) (layer Edge.Cuts) (width 0.15))

Commit message: Minor adjustments
Parts:
- moved J1 0.63 mm to (121.9, 76.8)
Other:
- outline, holes or cut-outs redrawn
Changed lines of the file:
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@@
   )
   (module Connector_Molex:Molex_KK-254_AE-6410-09A_1x09_P2.54mm_Vertical (layer F.Cu)
-    (at 121.92 76.2 180)
+    (at 121.92 76.835 180)
     (descr "Molex KK-254 Interconnect System, old/engineering part number: AE-6410-09A example for new part number: 22-27-2091, 9 Pins (http://www.molex.com/pdm_docs/sd/022272021_sd.pdf), generated with kicad-footprint-generator")
     (tags "connector Molex KK-254 side entry")
@@
     )
   )
-  (gr_line (start 99.695 72.39) (end 99.695 80.01) (layer F.SilkS) (width 0.2))
-  (gr_line (start 123.825 72.39) (end 99.695 72.39) (layer F.SilkS) (width 0.2))
+  (gr_line (start 99.695 73.025) (end 99.695 80.645) (layer F.SilkS) (width 0.2))
+  (gr_line (start 123.825 73.025) (end 99.695 73.025) (layer F.SilkS) (width 0.2))
   (gr_line (start 218.44 49.53) (end 218.44 57.15) (layer F.SilkS) (width 0.15))
   (gr_line (start 226.06 49.53) (end 218.44 49.53) (layer F.SilkS) (width 0.15))
@@
   (gr_line (start 73.025 57.15) (end 73.025 64.77) (layer F.SilkS) (width 0.15))
   (gr_line (start 80.645 57.15) (end 73.025 57.15) (layer F.SilkS) (width 0.15))
-  (gr_circle (center 144.145 57.785) (end 145.632898 59.055) (layer Edge.Cuts) (width 0.15))
-  (gr_circle (center 90.17 59.69) (end 91.657898 60.96) (layer Edge.Cuts) (width 0.15))
-  (gr_circle (center 144.145 64.135) (end 145.632898 65.405) (layer Edge.Cuts) (width 0.15))
-  (gr_circle (center 198.12 68.58) (end 199.607898 69.85) (layer Edge.Cuts) (width 0.15))
+  (gr_circle (center 144.399 57.785) (end 145.886898 59.055) (layer Edge.Cuts) (width 0.15))
+  (gr_circle (center 90.424 59.69) (end 91.911898 60.96) (layer Edge.Cuts) (width 0.15))
+  (gr_circle (center 144.399 64.135) (end 145.886898 65.405) (layer Edge.Cuts) (width 0.15))
+  (gr_circle (center 198.374 68.58) (end 199.861898 69.85) (layer Edge.Cuts) (width 0.15))
   (gr_line (start 67.277387 134.230068) (end 229.837387 134.230068) (layer Edge.Cuts) (width 0.15))
   (gr_line (start 67.277387 108.830068) (end 213.327387 108.830068) (layer Edge.Cuts) (width 0.15))

Commit message: Minor adjustments
Parts:
- moved D7 2.54 mm to (76.8, 57.1)
- moved D6 2.03 mm to (103.9, 60.2)
- moved D1 1.91 mm to (222.2, 50.2)
- moved D5 1.52 mm to (130.9, 63.2)
- moved D4 1.02 mm to (158.0, 66.3)
- moved D3 0.51 mm to (185.0, 69.3)
Other:
- outline, holes or cut-outs redrawn

Commit message: Minor adjustments
Parts:
- moved D2 5.00 mm to (212.1, 67.4)
- moved D3 4.00 mm to (185.1, 65.3)
- moved D1 3.61 mm to (225.2, 52.2)
- moved D4 3.00 mm to (158.0, 63.3)
- moved D5 2.00 mm to (131.0, 61.2)
- moved D6 1.00 mm to (103.9, 59.2)
Changed lines of the file:
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@@
   )
   (module LED_THT:LED_D5.0mm_Clear (layer F.Cu)
-    (at 103.886 60.198 270)
+    (at 103.895 59.198 270)
     (descr "LED, diameter 5.0mm, 2 pins, http://cdn-reichelt.de/documents/datenblatt/A500/LL-504BC2E-009.pdf")
     (tags "LED diameter 5.0mm 2 pins")
@@
   )
   (module LED_THT:LED_D5.0mm_Clear (layer F.Cu)
-    (at 130.937 63.246 270)
+    (at 130.955 61.246 270)
     (descr "LED, diameter 5.0mm, 2 pins, http://cdn-reichelt.de/documents/datenblatt/A500/LL-504BC2E-009.pdf")
     (tags "LED diameter 5.0mm 2 pins")
@@
   )
   (module LED_THT:LED_D5.0mm_Clear (layer F.Cu)
-    (at 157.988 66.294 270)
+    (at 158.015 63.294 270)
     (descr "LED, diameter 5.0mm, 2 pins, http://cdn-reichelt.de/documents/datenblatt/A500/LL-504BC2E-009.pdf")
     (tags "LED diameter 5.0mm 2 pins")
@@
   )
   (module LED_THT:LED_D5.0mm_Clear (layer F.Cu)
-    (at 185.039 69.342 270)
+    (at 185.075 65.342 270)
     (descr "LED, diameter 5.0mm, 2 pins, http://cdn-reichelt.de/documents/datenblatt/A500/LL-504BC2E-009.pdf")
     (tags "LED diameter 5.0mm 2 pins")
@@
   )
   (module LED_THT:LED_D5.0mm_Clear (layer F.Cu)
-    (at 212.09 72.39 270)
+    (at 212.135 67.39 270)
     (descr "LED, diameter 5.0mm, 2 pins, http://cdn-reichelt.de/documents/datenblatt/A500/LL-504BC2E-009.pdf")
     (tags "LED diameter 5.0mm 2 pins")
@@
   )
   (module LED_THT:LED_D5.0mm_Clear (layer F.Cu)
-    (at 222.25 50.165 270)
+    (at 225.25 52.165 270)
     (descr "LED, diameter 5.0mm, 2 pins, http://cdn-reichelt.de/documents/datenblatt/A500/LL-504BC2E-009.pdf")
     (tags "LED diameter 5.0mm 2 pins")

Commit message: Minor adjustments
Parts:
- moved D2 4.90 mm to (212.1, 72.3)
- moved D3 3.90 mm to (185.1, 69.2)
- moved D1 3.61 mm to (222.2, 50.2)
- moved D4 2.90 mm to (158.0, 66.2)
- moved D5 1.90 mm to (131.0, 63.1)
- moved D6 0.90 mm to (103.9, 60.1)
- moved D7 0.10 mm to (76.8, 57.0)
Changed lines of the file:
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@@
   )
   (module LED_THT:LED_D5.0mm_Clear (layer F.Cu)
-    (at 76.835 57.15 270)
+    (at 76.835 57.05 270)
     (descr "LED, diameter 5.0mm, 2 pins, http://cdn-reichelt.de/documents/datenblatt/A500/LL-504BC2E-009.pdf")
     (tags "LED diameter 5.0mm 2 pins")
@@
   )
   (module LED_THT:LED_D5.0mm_Clear (layer F.Cu)
-    (at 103.895 59.198 270)
+    (at 103.895 60.098 270)
     (descr "LED, diameter 5.0mm, 2 pins, http://cdn-reichelt.de/documents/datenblatt/A500/LL-504BC2E-009.pdf")
     (tags "LED diameter 5.0mm 2 pins")
@@
   )
   (module LED_THT:LED_D5.0mm_Clear (layer F.Cu)
-    (at 130.955 61.246 270)
+    (at 130.955 63.146 270)
     (descr "LED, diameter 5.0mm, 2 pins, http://cdn-reichelt.de/documents/datenblatt/A500/LL-504BC2E-009.pdf")
     (tags "LED diameter 5.0mm 2 pins")
@@
   )
   (module LED_THT:LED_D5.0mm_Clear (layer F.Cu)
-    (at 158.015 63.294 270)
+    (at 158.015 66.194 270)
     (descr "LED, diameter 5.0mm, 2 pins, http://cdn-reichelt.de/documents/datenblatt/A500/LL-504BC2E-009.pdf")
     (tags "LED diameter 5.0mm 2 pins")
@@
   )
   (module LED_THT:LED_D5.0mm_Clear (layer F.Cu)
-    (at 185.075 65.342 270)
+    (at 185.075 69.242 270)
     (descr "LED, diameter 5.0mm, 2 pins, http://cdn-reichelt.de/documents/datenblatt/A500/LL-504BC2E-009.pdf")
     (tags "LED diameter 5.0mm 2 pins")
@@
   )
   (module LED_THT:LED_D5.0mm_Clear (layer F.Cu)
-    (at 212.135 67.39 270)
+    (at 212.135 72.29 270)
     (descr "LED, diameter 5.0mm, 2 pins, http://cdn-reichelt.de/documents/datenblatt/A500/LL-504BC2E-009.pdf")
     (tags "LED diameter 5.0mm 2 pins")
@@
   )
   (module LED_THT:LED_D5.0mm_Clear (layer F.Cu)
-    (at 225.25 52.165 270)
+    (at 222.25 50.165 270)
     (descr "LED, diameter 5.0mm, 2 pins, http://cdn-reichelt.de/documents/datenblatt/A500/LL-504BC2E-009.pdf")
     (tags "LED diameter 5.0mm 2 pins")
@@
   (gr_line (start 218.44 47.625) (end 218.44 55.245) (layer F.SilkS) (width 0.15))
   (gr_line (start 226.06 47.625) (end 218.44 47.625) (layer F.SilkS) (width 0.15))
-  (gr_line (start 208.28 69.85) (end 208.28 77.47) (layer F.SilkS) (width 0.15))
-  (gr_line (start 215.9 69.85) (end 208.28 69.85) (layer F.SilkS) (width 0.15))
-  (gr_line (start 181.229 66.802) (end 181.229 74.422) (layer F.SilkS) (width 0.15))
-  (gr_line (start 188.849 66.802) (end 181.229 66.802) (layer F.SilkS) (width 0.15))
-  (gr_line (start 154.178 63.754) (end 154.178 71.374) (layer F.SilkS) (width 0.15))
-  (gr_line (start 161.798 63.754) (end 154.178 63.754) (layer F.SilkS) (width 0.15))
-  (gr_line (start 127.127 60.706) (end 127.127 68.326) (layer F.SilkS) (width 0.15))
-  (gr_line (start 134.747 60.706) (end 127.127 60.706) (layer F.SilkS) (width 0.15))
-  (gr_line (start 100.076 57.658) (end 100.076 65.278) (layer F.SilkS) (width 0.15))
-  (gr_line (start 107.696 57.658) (end 100.076 57.658) (layer F.SilkS) (width 0.15))
-  (gr_line (start 73.025 54.61) (end 73.025 62.23) (layer F.SilkS) (width 0.15))
-  (gr_line (start 80.645 54.61) (end 73.025 54.61) (layer F.SilkS) (width 0.15))
+  (gr_line (start 208.325 69.85) (end 208.325 77.47) (layer F.SilkS) (width 0.15))
+  (gr_line (start 215.945 69.85) (end 208.325 69.85) (layer F.SilkS) (width 0.15))
+  (gr_line (start 181.265 66.702) (end 181.265 74.322) (layer F.SilkS) (width 0.15))
+  (gr_line (start 188.885 66.702) (end 181.265 66.702) (layer F.SilkS) (width 0.15))
+  (gr_line (start 154.205 63.654) (end 154.205 71.274) (layer F.SilkS) (width 0.15))
+  (gr_line (start 161.825 63.654) (end 154.205 63.654) (layer F.SilkS) (width 0.15))
+  (gr_line (start 127.145 60.606) (end 127.145 68.226) (layer F.SilkS) (width 0.15))
+  (gr_line (start 134.765 60.606) (end 127.145 60.606) (layer F.SilkS) (width 0.15))
+  (gr_line (start 100.085 57.558) (end 100.085 65.178) (layer F.SilkS) (width 0.15))
+  (gr_line (start 107.705 57.558) (end 100.085 57.558) (layer F.SilkS) (width 0.15))
+  (gr_line (start 73.025 54.51) (end 73.025 62.13) (layer F.SilkS) (width 0.15))
+  (gr_line (start 80.645 54.51) (end 73.025 54.51) (layer F.SilkS) (width 0.15))
   (gr_circle (center 144.907 57.277) (end 146.394898 58.547) (layer Edge.Cuts) (width 0.15))
   (gr_circle (center 90.424 57.785) (end 91.911898 59.055) (layer Edge.Cuts) (width 0.15))

Commit message: Minor adjustments
Parts:
- moved D2 0.06 mm to (212.2, 72.3)

Commit message: Minor adjustments
Parts:
- moved D1 1.50 mm to (222.2, 51.7)
Other:
- board text added: "v1.11"
Changed lines of the file:
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@@
   (general
     (thickness 1.6)
-    (drawings 30)
+    (drawings 31)
     (tracks 0)
     (zones 0)
@@
     (solder_mask_min_width 0.25)
     (aux_axis_origin 0 0)
-    (visible_elements FFFFFF7F)
+    (visible_elements FFFFEF7F)
     (pcbplotparams
       (layerselection 0x010fc_ffffffff)
@@
   )
   (module LED_THT:LED_D5.0mm_Clear (layer F.Cu)
-    (at 76.835 57.05 270)
+    (at 76.83 57.05 270)
     (descr "LED, diameter 5.0mm, 2 pins, http://cdn-reichelt.de/documents/datenblatt/A500/LL-504BC2E-009.pdf")
     (tags "LED diameter 5.0mm 2 pins")
@@
   )
   (module LED_THT:LED_D5.0mm_Clear (layer F.Cu)
-    (at 103.906 60.098 270)
+    (at 103.901 60.098 270)
     (descr "LED, diameter 5.0mm, 2 pins, http://cdn-reichelt.de/documents/datenblatt/A500/LL-504BC2E-009.pdf")
     (tags "LED diameter 5.0mm 2 pins")
@@
   )
   (module LED_THT:LED_D5.0mm_Clear (layer F.Cu)
-    (at 130.977 63.146 270)
+    (at 130.972 63.146 270)
     (descr "LED, diameter 5.0mm, 2 pins, http://cdn-reichelt.de/documents/datenblatt/A500/LL-504BC2E-009.pdf")
     (tags "LED diameter 5.0mm 2 pins")
@@
   )
   (module LED_THT:LED_D5.0mm_Clear (layer F.Cu)
-    (at 158.048 66.194 270)
+    (at 158.043 66.194 270)
     (descr "LED, diameter 5.0mm, 2 pins, http://cdn-reichelt.de/documents/datenblatt/A500/LL-504BC2E-009.pdf")
     (tags "LED diameter 5.0mm 2 pins")
@@
   )
   (module LED_THT:LED_D5.0mm_Clear (layer F.Cu)
-    (at 185.119 69.242 270)
+    (at 185.114 69.242 270)
     (descr "LED, diameter 5.0mm, 2 pins, http://cdn-reichelt.de/documents/datenblatt/A500/LL-504BC2E-009.pdf")
     (tags "LED diameter 5.0mm 2 pins")
@@
   )
   (module LED_THT:LED_D5.0mm_Clear (layer F.Cu)
-    (at 212.19 72.29 270)
+    (at 212.185 72.29 270)
     (descr "LED, diameter 5.0mm, 2 pins, http://cdn-reichelt.de/documents/datenblatt/A500/LL-504BC2E-009.pdf")
     (tags "LED diameter 5.0mm 2 pins")
@@
   )
   (module LED_THT:LED_D5.0mm_Clear (layer F.Cu)
-    (at 222.25 50.165 270)
+    (at 222.25 51.665 270)
     (descr "LED, diameter 5.0mm, 2 pins, http://cdn-reichelt.de/documents/datenblatt/A500/LL-504BC2E-009.pdf")
     (tags "LED diameter 5.0mm 2 pins")
@@
     )
   )
+  (gr_text v1.11 (at 272.02 193.09) (layer F.Cu)
+    (effects (font (size 1.5 1.5) (thickness 0.3)))
+  )
   (gr_line (start 99.695 73.025) (end 99.695 80.645) (layer F.SilkS) (width 0.2))
   (gr_line (start 123.825 73.025) (end 99.695 73.025) (layer F.SilkS) (width 0.2))
-  (gr_line (start 218.44 47.625) (end 218.44 55.245) (layer F.SilkS) (width 0.15))
-  (gr_line (start 226.06 47.625) (end 218.44 47.625) (layer F.SilkS) (width 0.15))
-  (gr_line (start 208.38 69.85) (end 208.38 77.47) (layer F.SilkS) (width 0.15))
-  (gr_line (start 216 69.85) (end 208.38 69.85) (layer F.SilkS) (width 0.15))
-  (gr_line (start 181.309 66.702) (end 181.309 74.322) (layer F.SilkS) (width 0.15))
-  (gr_line (start 188.929 66.702) (end 181.309 66.702) (layer F.SilkS) (width 0.15))
-  (gr_line (start 154.238 63.654) (end 154.238 71.274) (layer F.SilkS) (width 0.15))
-  (gr_line (start 161.858 63.654) (end 154.238 63.654) (layer F.SilkS) (width 0.15))
-  (gr_line (start 127.167 60.606) (end 127.167 68.226) (layer F.SilkS) (width 0.15))
-  (gr_line (start 134.787 60.606) (end 127.167 60.606) (layer F.SilkS) (width 0.15))
-  (gr_line (start 100.096 57.558) (end 100.096 65.178) (layer F.SilkS) (width 0.15))
-  (gr_line (start 107.716 57.558) (end 100.096 57.558) (layer F.SilkS) (width 0.15))
-  (gr_line (start 73.025 54.51) (end 73.025 62.13) (layer F.SilkS) (width 0.15))
-  (gr_line (start 80.645 54.51) (end 73.025 54.51) (layer F.SilkS) (width 0.15))
+  (gr_line (start 218.44 49.125) (end 218.44 56.745) (layer F.SilkS) (width 0.15))
+  (gr_line (start 226.06 49.125) (end 218.44 49.125) (layer F.SilkS) (width 0.15))
+  (gr_line (start 208.375 69.85) (end 208.375 77.47) (layer F.SilkS) (width 0.15))
+  (gr_line (start 215.995 69.85) (end 208.375 69.85) (layer F.SilkS) (width 0.15))
+  (gr_line (start 181.304 66.702) (end 181.304 74.322) (layer F.SilkS) (width 0.15))
+  (gr_line (start 188.924 66.702) (end 181.304 66.702) (layer F.SilkS) (width 0.15))
+  (gr_line (start 154.233 63.654) (end 154.233 71.274) (layer F.SilkS) (width 0.15))
+  (gr_line (start 161.853 63.654) (end 154.233 63.654) (layer F.SilkS) (width 0.15))
+  (gr_line (start 127.162 60.606) (end 127.162 68.226) (layer F.SilkS) (width 0.15))
+  (gr_line (start 134.782 60.606) (end 127.162 60.606) (layer F.SilkS) (width 0.15))
+  (gr_line (start 100.091 57.558) (end 100.091 65.178) (layer F.SilkS) (width 0.15))
+  (gr_line (start 107.711 57.558) (end 100.091 57.558) (layer F.SilkS) (width 0.15))
+  (gr_line (start 73.02 54.51) (end 73.02 62.13) (layer F.SilkS) (width 0.15))
+  (gr_line (start 80.64 54.51) (end 73.02 54.51) (layer F.SilkS) (width 0.15))
   (gr_circle (center 144.907 57.277) (end 146.394898 58.547) (layer Edge.Cuts) (width 0.15))
   (gr_circle (center 90.424 57.785) (end 91.911898 59.055) (layer Edge.Cuts) (width 0.15))

Commit message: Minor adjustments
Parts:
- moved D1 1.50 mm to (222.2, 53.2)
Other:
- outline, holes or cut-outs redrawn
- board text added: "Rev: v1.12"
- board text removed: "v1.11"
Changed lines of the file:
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@@
   )
   (page A4)
+  (title_block
+    (rev v1.12)
+  )
   (layers
     (0 F.Cu signal)
@@
   )
   (module LED_THT:LED_D5.0mm_Clear (layer F.Cu)
-    (at 222.25 51.665 270)
+    (at 222.25 53.165 270)
     (descr "LED, diameter 5.0mm, 2 pins, http://cdn-reichelt.de/documents/datenblatt/A500/LL-504BC2E-009.pdf")
     (tags "LED diameter 5.0mm 2 pins")
@@
     )
   )
-  (gr_text v1.11 (at 272.02 193.09) (layer F.Cu)
-    (effects (font (size 1.5 1.5) (thickness 0.3)))
+  (gr_text "Rev: v1.12" (at 68.81 81.1) (layer F.SilkS)
+    (effects (font (size 1.5 1.5) (thickness 0.3)) (justify left))
   )
   (gr_line (start 99.695 73.025) (end 99.695 80.645) (layer F.SilkS) (width 0.2))
   (gr_line (start 123.825 73.025) (end 99.695 73.025) (layer F.SilkS) (width 0.2))
-  (gr_line (start 218.44 49.125) (end 218.44 56.745) (layer F.SilkS) (width 0.15))
-  (gr_line (start 226.06 49.125) (end 218.44 49.125) (layer F.SilkS) (width 0.15))
+  (gr_line (start 218.44 50.625) (end 218.44 58.245) (layer F.SilkS) (width 0.15))
+  (gr_line (start 226.06 50.625) (end 218.44 50.625) (layer F.SilkS) (width 0.15))
   (gr_line (start 208.375 69.85) (end 208.375 77.47) (layer F.SilkS) (width 0.15))
   (gr_line (start 215.995 69.85) (end 208.375 69.85) (layer F.SilkS) (width 0.15))
@@
   (gr_line (start 73.02 54.51) (end 73.02 62.13) (layer F.SilkS) (width 0.15))
   (gr_line (start 80.64 54.51) (end 73.02 54.51) (layer F.SilkS) (width 0.15))
-  (gr_circle (center 144.907 57.277) (end 146.394898 58.547) (layer Edge.Cuts) (width 0.15))
+  (gr_circle (center 144.407 57.277) (end 145.894898 58.547) (layer Edge.Cuts) (width 0.15))
   (gr_circle (center 90.424 57.785) (end 91.911898 59.055) (layer Edge.Cuts) (width 0.15))
-  (gr_circle (center 144.907 63.627) (end 146.394898 64.897) (layer Edge.Cuts) (width 0.15))
-  (gr_circle (center 199.644 69.85) (end 201.131898 71.12) (layer Edge.Cuts) (width 0.15))
+  (gr_circle (center 144.407 63.627) (end 145.894898 64.897) (layer Edge.Cuts) (width 0.15))
+  (gr_circle (center 199.144 69.85) (end 200.631898 71.12) (layer Edge.Cuts) (width 0.15))
   (gr_line (start 67.277387 134.230068) (end 229.837387 134.230068) (layer Edge.Cuts) (width 0.15))
   (gr_line (start 67.277387 108.830068) (end 213.327387 108.830068) (layer Edge.Cuts) (width 0.15))
